Commit message: Feat: Add xacro and STL files for robot visualization

File: remote_node/urdf/swiftpro.xacro (robot description, xacro)
@@ -10,5 +10,5 @@
 	<visual>
 		<geometry>
-			<mesh filename="package://swiftpro/urdf/pro_links/Base.STL"/>
+			<mesh filename="package://remote_node/urdf/Base.STL"/>
 		</geometry>
 		<origin xyz = "0 0 0 " rpy = "0 0 0"/>
@@ -27,5 +27,5 @@
 	<visual>
 		<geometry>
-			<mesh filename="package://swiftpro/urdf/pro_links/Link1.STL"/>
+			<mesh filename="package://remote_node/urdf/Link1.STL"/>
 		</geometry>
 		<origin xyz = "0 0 -0.0723" rpy = "0 0 0" />
@@ -51,5 +51,5 @@
 	<visual>
 		<geometry>
-			<mesh filename="package://swiftpro/urdf/pro_links/Link2.STL"/>
+			<mesh filename="package://remote_node/urdf/Link2.STL"/>
 		</geometry>
 		<origin xyz = "-0.0132 0 -0.1056" rpy = "0 0 0" />
@@ -75,5 +75,5 @@
 	<visual>
 		<geometry>
-			<mesh filename="package://swiftpro/urdf/pro_links/Link3.STL"/>
+			<mesh filename="package://remote_node/urdf/Link3.STL"/>
 		</geometry>
 		<origin xyz="-0.0132 0 -0.24767"/>
@@ -99,5 +99,5 @@
 	<visual>
 		<geometry>
-			<mesh filename="package://swiftpro/urdf/pro_links/Link4.STL"/>
+			<mesh filename="package://remote_node/urdf/Link4.STL"/>
 		</geometry>
 		<origin xyz = "-0.0132 0 -0.24767" rpy = "0 0 0" />
@@ -123,5 +123,5 @@
 	<visual>
 		<geometry>
-			<mesh filename="package://swiftpro/urdf/pro_links/Link5.STL"/>
+			<mesh filename="package://remote_node/urdf/Link5.STL"/>
 		</geometry>
 		<origin xyz = "0.0215 0 -0.1223" rpy = "0 0 0" />
@@ -147,5 +147,5 @@
 	<visual>
 		<geometry>
-			<mesh filename="package://swiftpro/urdf/pro_links/Link6.STL"/>
+			<mesh filename="package://remote_node/urdf/Link6.STL"/>
 		</geometry>
 		<origin xyz = "-0.0132 0 -0.1056" rpy = "0 0 0" />
@@ -171,5 +171,5 @@
 	<visual>
 		<geometry>
-			<mesh filename="package://swiftpro/urdf/pro_links/Link7.STL"/>
+			<mesh filename="package://remote_node/urdf/Link7.STL"/>
 		</geometry>
 		<origin xyz = "0.0323 0 -0.10258" rpy = "0 0 0" />
@@ -195,5 +195,5 @@
 	<visual>
 		<geometry>
-			<mesh filename="package://swiftpro/urdf/pro_links/Gripper.STL"/>
+			<mesh filename="package://remote_node/urdf/Gripper.STL"/>
 		</geometry>
 		<origin xyz = "-0.17201 0 -0.24651" rpy = "0 0 0" />
@@ -219,5 +219,5 @@
 	<visual>
 		<geometry>
-			<mesh filename="package://swiftpro/urdf/pro_links/Link9.STL"/>
+			<mesh filename="package://remote_node/urdf/Link9.STL"/>
 		</geometry>
 		<origin xyz = "-0.19941 0 -0.27471" rpy = "0 0 0" />

Commit message: feat: Get RViz working with our generated URDF doc: update README

File: remote_node/urdf/swiftpro.xacro (robot description, xacro)
@@ -1,4 +1,11 @@
 <?xml version="1.0"?>
 <robot xmlns:xacro="http://www.ros.org/wiki/xacro" name="swiftpro" >
+<!-- Dummy root link without inertia -->
+<!-- mitigates :
+    [robot_state_publisher-1] [WARN] [1738930205.934000376] [kdl_parser]: The root link Base
+	 has an inertia specified in the URDF, but KDL does not support a root link with an inertia.
+	 As a workaround, you can add an extra dummy link to your URDF.
+-->
+<link name="dummy_base"/>
 <link name="Base">
 	<inertial>
@@ -18,4 +25,10 @@
     </visual>
 </link>
+ <!-- Fixed joint between dummy_base and Base -->
+    <joint name="dummy_base_to_base" type="fixed">
+        <parent link="dummy_base"/>
+        <child link="Base"/>
+        <origin xyz="0 0 0" rpy="0 0 0"/>
+    </joint>
 <link name="Link1">
 	<inertial>
