Commit message: Major refactor: correct kinematics, two-image container design, remove swiftpro_control
- swiftpro.xacro: add <mimic> joints for all parallel linkage constraints,
  verified on physical hardware. Joint8 mimics Joint3 x-1.0 (not Joint2).
  Joint9 changed to fixed. Realistic joint limits on driven joints.

- swiftpro_hardware: add missing <thread> <mutex> <cmath> includes, extract
  DRIVEN_JOINT_NAMES and DEG_TO_RAD constants, clarify publish_state comments,
  fix instance_ = nullptr in destructor, const-correct service handlers

- swiftpro_kinematics: complete rewrite as analytical FK node. Removed TF
  broadcasting (robot_state_publisher owns TF). Now publishes Cartesian end
  effector position on /swiftpro/end_effector_position. Geometric FK from
  first principles with inline documentation.

- swiftpro_kinematics/CMakeLists.txt: add missing ament_cmake, remove tf2/tf2_ros
  dependencies (no longer needed)

- swiftpro_resources/CMakeLists.txt: fix ament_cmake_cpplint duplicate registration

- swiftpro_control: deleted — placeholder with no purpose. Hardware node services
  cover all needed control operations directly.

- Dockerfile: lean dev image — remove source baking and rosdep, add clangd,
  robot-state-publisher, tf2, tf2-ros. Add /opt/topicfs_typesupport directory.

- Dockerfile.runtime: rebase on ros:jazzy-ros-core, remove all dev tools,
  runtime dependencies only, no baked binaries or entrypoint

- docker-compose.yml: add userns_mode keep-id (fixes file ownership in container),
  mount full workspace as /swiftros_ws, remove ulimits (not permitted on NUC),
  remove /dev mount (not needed for dev)

- docker-compose.runtime.yml: new file for worker deployment via podman-compose

- entrypoint.sh: new runtime startup script, sources ROS2 + install overlay,
  clear error if artifacts not deployed, SWIFTPRO_PORT configurable via env

- README.md: complete rewrite documenting all nodes, kinematics, parallel linkage
  physics, two-image container design, registry, and deployment workflow

File: swiftpro_resources/urdf/swiftpro.xacro (robot description, xacro)
@@ -1,249 +1,317 @@
 <?xml version="1.0"?>
-<robot xmlns:xacro="http://www.ros.org/wiki/xacro" name="swiftpro" >
-<!-- Dummy root link without inertia -->
-<!-- mitigates :
-    [robot_state_publisher-1] [WARN] [1738930205.934000376] [kdl_parser]: The root link Base
-	 has an inertia specified in the URDF, but KDL does not support a root link with an inertia.
-	 As a workaround, you can add an extra dummy link to your URDF.
+<!-- swiftpro.xacro -->
+<!-- Copyright 2025 Jack Sidman Smith -->
+<!-- Licensed under the MIT License. See LICENSE in project root. -->
+<!--
+  UArm Swift Pro URDF with parallel linkage constraints.
+  The arm has 3 physical servos:
+    Joint1 — base rotation       (servo 0)  Z axis
+    Joint2 — shoulder elevation  (servo 1)  Y axis
+    Joint3 — elbow/forearm       (servo 2)  Y axis
+  All other joints are mechanically constrained by the parallel linkage
+  and expressed as <mimic> joints. robot_state_publisher computes and
+  broadcasts their values automatically from Joint1/2/3.
+  The hardware node (swiftpro_hardware) publishes JointState for
+  Joint1, Joint2, Joint3 only.
+  Parallel linkage geometry — two four-bar loops:
+  Loop 1 — upper arm parallelogram:
+    Link2  (Joint2) — upper arm front rod      — driven by servo 1
+    Link5  (Joint5) — upper arm rear rod       — mimics Joint2 × -1.0
+    Link4  (Joint4) — triangular connector     — mimics Joint3 × +1.0
+    The triangle (Link4) transfers elbow rotation to the wrist chain.
+    Shoulder movement is fully cancelled within this loop — it never
+    reaches the end effector.
+  Loop 2 — wrist parallelogram:
+    Link6  (Joint6) — wrist rear upper         — mimics Joint2 × +1.0
+    Link7  (Joint7) — wrist rear lower         — mimics Joint3 × +1.0
+    Link8  (Joint8) — end effector mount       — mimics Joint3 × -1.0
+    Only elbow rotation (Joint3) reaches the end effector.
+    Joint8 cancels it to keep the gripper level.
+  Verified against physical hardware:
+    - Moving shoulder only: forearm links stay parallel ✓
+    - Moving elbow only:    upper arm links stay parallel ✓
+    - Joint8 compensation source is Joint3, not Joint2 ✓
+  Joint9 is fixed — the gripper jaw is not servo-driven in the
+  base UArm Swift Pro configuration.
 -->
+<robot xmlns:xacro="http://www.ros.org/wiki/xacro" name="swiftpro">
+<!-- ============================================================ -->
+<!-- Dummy root — avoids KDL inertia warning on root link         -->
+<!-- ============================================================ -->
 <link name="dummy_base"/>
+<joint name="dummy_base_to_base" type="fixed">
+  <parent link="dummy_base"/>
+  <child link="Base"/>
+  <origin xyz="0 0 0" rpy="0 0 0"/>
+</joint>
+<!-- ============================================================ -->
+<!-- Base                                                          -->
+<!-- ============================================================ -->
 <link name="Base">
-	<inertial>
-		<origin xyz="0.010476 0.000747 0.035226" rpy="0 0 0"/>
-		<mass value="1.886"/>
-		<inertia ixx="0.001196219" ixy="-0.000029358" ixz="0.000014859"
-				 iyy="0.001147997" iyz="0.000016274"  izz="0.001425617"/>
-	</inertial>
-	<visual>
-		<geometry>
-			<mesh filename="package://swiftpro_resources/urdf/Base.STL"/>
-		</geometry>
-		<origin xyz = "0 0 0 " rpy = "0 0 0"/>
-		<material name = "">
-			<color rgba = "0.3 0.3 0.3 1" />
-		</material>
-    </visual>
-</link>
- <!-- Fixed joint between dummy_base and Base -->
-    <joint name="dummy_base_to_base" type="fixed">
-        <parent link="dummy_base"/>
-        <child link="Base"/>
-        <origin xyz="0 0 0" rpy="0 0 0"/>
-    </joint>
+  <inertial>
+    <origin xyz="0.010476 0.000747 0.035226" rpy="0 0 0"/>
+    <mass value="1.886"/>
+    <inertia ixx="0.001196219" ixy="-0.000029358" ixz="0.000014859"
+             iyy="0.001147997" iyz="0.000016274"  izz="0.001425617"/>
+  </inertial>
+  <visual>
+    <geometry>
+      <mesh filename="package://swiftpro_resources/urdf/Base.STL"/>
+    </geometry>
+    <origin xyz="0 0 0" rpy="0 0 0"/>
+    <material name="dark_grey">
+      <color rgba="0.3 0.3 0.3 1"/>
+    </material>
+  </visual>
+</link>
+<!-- ============================================================ -->
+<!-- Link1 — base turntable                                        -->
+<!-- Joint1 — base rotation (Z axis) — SERVO 0                    -->
+<!-- ============================================================ -->
 <link name="Link1">
-	<inertial>
-		<origin xyz="-0.002175 0 0.029097" rpy="0 0 0"/>
-		<mass value="0.2141"/>
-		<inertia ixx="0.000496945" ixy="-0.000000082" ixz="-0.000002744"
-				 iyy="0.000150389" iyz="-0.000000002" izz="0.000522487"/>
-	</inertial>
-	<visual>
-		<geometry>
-			<mesh filename="package://swiftpro_resources/urdf/Link1.STL"/>
-		</geometry>
-		<origin xyz = "0 0 -0.0723" rpy = "0 0 0" />
-		<material name = "">
-			<color rgba = "0.3 0.3 0.3 1" />
-		</material>
-    </visual>
+  <inertial>
+    <origin xyz="-0.002175 0 0.029097" rpy="0 0 0"/>
+    <mass value="0.2141"/>
+    <inertia ixx="0.000496945" ixy="-0.000000082" ixz="-0.000002744"
+             iyy="0.000150389" iyz="-0.000000002" izz="0.000522487"/>
+  </inertial>
+  <visual>
+    <geometry>
+      <mesh filename="package://swiftpro_resources/urdf/Link1.STL"/>
+    </geometry>
+    <origin xyz="0 0 -0.0723" rpy="0 0 0"/>
+    <material name="dark_grey"/>
+  </visual>
 </link>
 <joint name="Joint1" type="revolute">
-	<axis xyz="0 0 1"/>
-	<limit effort = "1000.0" lower = "-3" upper = "3" velocity = "0" />
-    <parent link="Base"/>
-    <child link="Link1"/>
-	<origin xyz= "0 0 0.0723" rpy = " 0 0 0" />
-</joint>
+  <axis xyz="0 0 1"/>
+  <limit effort="1000.0" lower="-1.57" upper="1.57" velocity="2.0"/>
+  <parent link="Base"/>
+  <child link="Link1"/>
+  <origin xyz="0 0 0.0723" rpy="0 0 0"/>
+</joint>
+<!-- ============================================================ -->
+<!-- Link2 — upper arm front rod                                   -->
+<!-- Joint2 — shoulder elevation (Y axis) — SERVO 1               -->
+<!-- ============================================================ -->
 <link name="Link2">
-	<inertial>
-		<origin xyz="-0.001071 0.001101 0.053193" rpy="0 0 0"/>
-		<mass value="0.026"/>
-		<inertia ixx="0.000061744" ixy="-0.000000025" ixz="-0.000000763"
-				 iyy="0.000062096" iyz="-0.000001053" izz="0.000002942"/>
-	</inertial>
-	<visual>
-		<geometry>
-			<mesh filename="package://swiftpro_resources/urdf/Link2.STL"/>
-		</geometry>
-		<origin xyz = "-0.0132 0 -0.1056" rpy = "0 0 0" />
-		<material name = "">
-			<color rgba = "0.3 0.3 0.3 1" />
-		</material>
-    </visual>
+  <inertial>
+    <origin xyz="-0.001071 0.001101 0.053193" rpy="0 0 0"/>
+    <mass value="0.026"/>
+    <inertia ixx="0.000061744" ixy="-0.000000025" ixz="-0.000000763"
+             iyy="0.000062096" iyz="-0.000001053" izz="0.000002942"/>
+  </inertial>
+  <visual>
+    <geometry>
+      <mesh filename="package://swiftpro_resources/urdf/Link2.STL"/>
+    </geometry>
+    <origin xyz="-0.0132 0 -0.1056" rpy="0 0 0"/>
+    <material name="dark_grey"/>
+  </visual>
 </link>
 <joint name="Joint2" type="revolute">
-	<axis xyz="0 1 0"/>
-	<limit effort = "1000.0" lower = "-3" upper = "3" velocity = "0" />
-    <parent link="Link1"/>
-    <child link="Link2"/>
-	<origin xyz= "0.0132 0 0.0333" rpy = " 0 0 0" />
-</joint>
+  <axis xyz="0 1 0"/>
+  <limit effort="1000.0" lower="-1.57" upper="1.57" velocity="2.0"/>
+  <parent link="Link1"/>
+  <child link="Link2"/>
+  <origin xyz="0.0132 0 0.0333" rpy="0 0 0"/>
+</joint>
+<!-- ============================================================ -->
+<!-- Link3 — forearm                                               -->
+<!-- Joint3 — elbow (Y axis) — SERVO 2                            -->
+<!-- ============================================================ -->
 <link name="Link3">
-	<inertial>
-		<origin xyz="0.101948 -0.00022 0.011917" rpy="0 0 0"/>
-		<mass value="0.023"/>
-		<inertia ixx="0.000001982" ixy="0.000000483" ixz="-0.000005373"
-				 iyy="0.000081264" iyz="0.000000008" izz="0.000080538"/>
-	</inertial>
-	<visual>
-		<geometry>
-			<mesh filename="package://swiftpro_resources/urdf/Link3.STL"/>
-		</geometry>
-		<origin xyz="-0.0132 0 -0.24767"/>
-		<material name="">
-			<color rgba = "0.3 0.3 0.3 1" />
-		</material>
-	</visual>
+  <inertial>
+    <origin xyz="0.101948 -0.00022 0.011917" rpy="0 0 0"/>
+    <mass value="0.023"/>
+    <inertia ixx="0.000001982" ixy="0.000000483" ixz="-0.000005373"
+             iyy="0.000081264" iyz="0.000000008" izz="0.000080538"/>
+  </inertial>
+  <visual>
+    <geometry>
+      <mesh filename="package://swiftpro_resources/urdf/Link3.STL"/>
+    </geometry>
+    <origin xyz="-0.0132 0 -0.24767" rpy="0 0 0"/>
+    <material name="dark_grey"/>
+  </visual>
 </link>
 <joint name="Joint3" type="revolute">
-	<axis xyz="0 1 0"/>
-	<parent link="Link2" />
-	<child link="Link3" />
-	<limit effort="1000" lower="-1.45" upper="1.45" velocity="0"/>
-	<origin xyz="0 0 0.14207 " rpy="0 0 0"/>
-</joint>
+  <axis xyz="0 1 0"/>
+  <limit effort="1000.0" lower="-1.45" upper="1.45" velocity="2.0"/>
+  <parent link="Link2"/>
+  <child link="Link3"/>
+  <origin xyz="0 0 0.14207" rpy="0 0 0"/>
+</joint>
+<!-- ============================================================ -->
+<!-- Link4 — triangular connector                                  -->
+<!-- Joint4 — mimics Joint3 × +1.0                                -->
+<!-- Transfers elbow rotation to the wrist chain.                  -->
+<!-- Pivots at the same point as Joint3 on Link2.                  -->
+<!-- ============================================================ -->
 <link name="Link4">
-	<inertial>
-		<origin xyz="-0.00235 0.013618 0.015458" rpy="0 0 0"/>
-		<mass value="0.003"/>
-		<inertia ixx="0.000000316" ixy="0.000000001"  ixz="0.000000177"
-				 iyy="0.000001679" iyz="-0.000000007" izz="0.000001378"/>
-	</inertial>
-	<visual>
-		<geometry>
-			<mesh filename="package://swiftpro_resources/urdf/Link4.STL"/>
-		</geometry>
-		<origin xyz = "-0.0132 0 -0.24767" rpy = "0 0 0" />
-		<material name = "">
-			<color rgba = "0.3 0.3 0.3 1" />
-		</material>
-    </visual>
+  <inertial>
+    <origin xyz="-0.00235 0.013618 0.015458" rpy="0 0 0"/>
+    <mass value="0.003"/>
+    <inertia ixx="0.000000316" ixy="0.000000001" ixz="0.000000177"
+             iyy="0.000001679" iyz="-0.000000007" izz="0.000001378"/>
+  </inertial>
+  <visual>
+    <geometry>
+      <mesh filename="package://swiftpro_resources/urdf/Link4.STL"/>
+    </geometry>
+    <origin xyz="-0.0132 0 -0.24767" rpy="0 0 0"/>
+    <material name="dark_grey"/>
+  </visual>
 </link>
 <joint name="Joint4" type="revolute">
-	<axis xyz="0 1 0"/>
-	<limit effort = "1000.0" lower = "-3" upper = "3" velocity = "0" />
-    <parent link="Link2"/>
-    <child link="Link4"/>
-	<origin xyz= "0 0 0.14207" rpy = " 0 0 0" />
-</joint>
+  <axis xyz="0 1 0"/>
+  <limit effort="1000.0" lower="-3" upper="3" velocity="2.0"/>
+  <parent link="Link2"/>
+  <child link="Link4"/>
+  <origin xyz="0 0 0.14207" rpy="0 0 0"/>
+  <mimic joint="Joint3" multiplier="1.0" offset="0.0"/>
+</joint>
+<!-- ============================================================ -->
+<!-- Link5 — upper arm rear rod                                    -->
+<!-- Joint5 — mimics Joint2 × -1.0                                -->
+<!-- Closes the upper arm parallelogram loop.                      -->
+<!-- Pivots on Link1 below Joint2.                                 -->
+<!-- ============================================================ -->
 <link name="Link5">
-	<inertial>
-		<origin xyz="0.000287 0.0157 0.072444" rpy="0 0 0"/>
-		<mass value="0.003"/>
-		<inertia ixx="0.000004841" ixy="0.000000000" ixz="0.000000023"
-				 iyy="0.000004863" iyz="0.000000000" izz="0.000000023"/>
-	</inertial>
-	<visual>
-		<geometry>
-			<mesh filename="package://swiftpro_resources/urdf/Link5.STL"/>
-		</geometry>
-		<origin xyz = "0.0215 0 -0.1223" rpy = "0 0 0" />
-		<material name = "">
-			<color rgba = "0.3 0.3 0.3 1" />
-		</material>
-    </visual>
+  <inertial>
+    <origin xyz="0.000287 0.0157 0.072444" rpy="0 0 0"/>
+    <mass value="0.003"/>
+    <inertia ixx="0.000004841" ixy="0.000000000" ixz="0.000000023"
+             iyy="0.000004863" iyz="0.000000000" izz="0.000000023"/>
+  </inertial>
+  <visual>
+    <geometry>
+      <mesh filename="package://swiftpro_resources/urdf/Link5.STL"/>
+    </geometry>
+    <origin xyz="0.0215 0 -0.1223" rpy="0 0 0"/>
+    <material name="dark_grey"/>
+  </visual>
 </link>
 <joint name="Joint5" type="revolute">
-	<axis xyz="0 1 0"/>
-	<limit effort = "1000.0" lower = "-3" upper = "3" velocity = "0" />
-    <parent link="Link1"/>
-    <child link="Link5"/>
-	<origin xyz= "-0.0215 0 0.05001" rpy = " 0 0 0" />
-</joint>
+  <axis xyz="0 1 0"/>
+  <limit effort="1000.0" lower="-3" upper="3" velocity="2.0"/>
+  <parent link="Link1"/>
+  <child link="Link5"/>
+  <origin xyz="-0.0215 0 0.05001" rpy="0 0 0"/>
+  <mimic joint="Joint2" multiplier="-1.0" offset="0.0"/>
+</joint>
+<!-- ============================================================ -->
+<!-- Link6 — wrist rear upper rod                                  -->
+<!-- Joint6 — mimics Joint2 × +1.0                                -->
+<!-- Follows shoulder rotation to position the wrist chain.        -->
+<!-- ============================================================ -->
 <link name="Link6">
-	<inertial>
-		<origin xyz="-0.014 -0.01391 -0.001062" rpy="0 0 0"/>
-		<mass value="0.003"/>
-		<inertia ixx="0.000000074" ixy="-0.000000060" ixz="0.000000055"
-				 iyy="0.000000951" iyz="-0.000000004" izz="0.000000923"/>
-	</inertial>
-	<visual>
-		<geometry>
-			<mesh filename="package://swiftpro_resources/urdf/Link6.STL"/>
-		</geometry>
-		<origin xyz = "-0.0132 0 -0.1056" rpy = "0 0 0" />
-		<material name = "">
-			<color rgba = "0.3 0.3 0.3 1" />
-		</material>
-    </visual>
+  <inertial>
+    <origin xyz="-0.014 -0.01391 -0.001062" rpy="0 0 0"/>
+    <mass value="0.003"/>
+    <inertia ixx="0.000000074" ixy="-0.000000060" ixz="0.000000055"
+             iyy="0.000000951" iyz="-0.000000004" izz="0.000000923"/>
+  </inertial>
+  <visual>
+    <geometry>
+      <mesh filename="package://swiftpro_resources/urdf/Link6.STL"/>
+    </geometry>
+    <origin xyz="-0.0132 0 -0.1056" rpy="0 0 0"/>
+    <material name="dark_grey"/>
+  </visual>
 </link>
 <joint name="Joint6" type="revolute">
-	<axis xyz="0 1 0"/>
-	<limit effort = "1000.0" lower = "-3" upper = "3" velocity = "0" />
-    <parent link="Link1"/>
-    <child link="Link6"/>
-	<origin xyz= "0.0132 0 0.0333" rpy = " 0 0 0" />
-</joint>
+  <axis xyz="0 1 0"/>
+  <limit effort="1000.0" lower="-3" upper="3" velocity="2.0"/>
+  <parent link="Link1"/>
+  <child link="Link6"/>
+  <origin xyz="0.0132 0 0.0333" rpy="0 0 0"/>
+  <mimic joint="Joint2" multiplier="1.0" offset="0.0"/>
+</joint>
+<!-- ============================================================ -->
+<!-- Link7 — wrist rear lower rod                                  -->
+<!-- Joint7 — mimics Joint3 × +1.0                                -->
+<!-- Transfers elbow rotation through the wrist rear chain.        -->
+<!-- ============================================================ -->
 <link name="Link7">
-	<inertial>
-		<origin xyz="-0.001242 -0.013867 0.083246" rpy="0 0 0"/>
-		<mass value="0.003"/>
-		<inertia ixx="0.000007052" ixy="0.000000003" ixz="0.000000055"
-				 iyy="0.000007058" iyz="0.000000117" izz="0.000000039"/>
-	</inertial>
-	<visual>
-		<geometry>
-			<mesh filename="package://swiftpro_resources/urdf/Link7.STL"/>
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